Commit message: Update urdf xacro

File: solo12_description/urdf/solo12.urdf.xacro (robot description, xacro)
@@ -5,13 +5,27 @@
   xmlns:sensor="http://playerstage.sourceforge.net/gazebo/xmlschema/#sensor"
   xmlns:xacro="http://playerstage.sourceforge.net/gazebo/xmlschema/#interface">
+  <!-- Simulation control arguments -->
+  <xacro:arg name="prefix" default="" />
   <xacro:arg name="use_sim" default="true" />
+  <xacro:arg name="use_mock_hardware" default="false" />
+  <xacro:arg name="mock_sensor_commands" default="false" />
+  <xacro:arg name="sim_gazebo_classic" default="false" />
+  <xacro:arg name="sim_gazebo" default="false" />
+  <xacro:arg name="simulation_controllers" default="" />
   <xacro:property name="color_name" value="grey" />
   <xacro:property name="color" value="0.8 0.8 0.8" />
   <xacro:property name="opacity" value="1.0" />
   <xacro:property name="mesh_ext" value="stl" />
+  <!-- Include ROS2 control xacro file -->
   <xacro:include filename="solo12.ros2_control.xacro"/>
+  <!-- ROS2 control macro for solo robot -->
   <xacro:solo12_ros2_control
-    use_sim="$(arg use_sim)"/>
-  <!-- This file is based on: https://github.com/open-dynamic-robot-initiative/open_robot_actuator_hardware/blob/master/mechanics/quadruped_robot_12dof_v1/README.md#quadruped-robot-12dof-v1 -->
+    name="solo"
+    prefix="$(arg prefix)"
+    use_mock_hardware="$(arg use_mock_hardware)"
+    mock_sensor_commands="$(arg mock_sensor_commands)"
+    sim_gazebo_classic="$(arg sim_gazebo_classic)"
+    sim_gazebo="$(arg sim_gazebo)"/>
+  <!-- Base link configuration -->
   <link name="base_link">
     <!-- BASE LINK INERTIAL -->
@@ -29,6 +43,5 @@
         <origin xyz="0 0 0" rpy="0 0 0" />
         <geometry>
-      <!-- <box size="0.1 0.1 0.1"/>-->
-      <mesh filename="file://$(find solo12_description)/meshes/collision/base.${mesh_ext}"/>
+            <mesh filename="file://$(find solo12_description)/meshes/collision/base.${mesh_ext}"/>
         </geometry>
         <material name="${color_name}">
@@ -40,5 +53,5 @@
         <origin xyz="0 0 0" rpy="0 0 0" />
         <geometry>
-      <mesh filename="file://$(find solo12_description)/meshes/collision/base.${mesh_ext}"/>
+            <mesh filename="file://$(find solo12_description)/meshes/collision/base.${mesh_ext}"/>
         </geometry>
         <material name="${color_name}">
@@ -46,5 +59,5 @@
         </material>
     </collision>
-    <!-- Bullet specific paramters -->
+    <!-- Bullet specific parameters -->
     <contact>
       <lateral_friction value="1.0"/>
@@ -94,3 +107,25 @@
       color="${color}"
       opacity="${opacity}"/>
+  <!-- Gazebo simulation control: gazebo classic or ignition -->
+  <xacro:if value="$(arg sim_gazebo_classic)">
+    <!-- Gazebo classic plugins -->
+    <gazebo reference="base_link">
+    </gazebo>
+    <gazebo>
+      <plugin filename="libgazebo_ros2_control.so" name="gazebo_ros2_control">
+        <parameters>$(arg simulation_controllers)</parameters>
+      </plugin>
+    </gazebo>
+  </xacro:if>
+  <xacro:if value="$(arg sim_gazebo)">
+    <!-- Gazebo Ignition plugins -->
+    <gazebo reference="base_link">
+    </gazebo>
+    <gazebo>
+      <plugin filename="libign_ros2_control-system.so" name="ign_ros2_control::IgnitionROS2ControlPlugin">
+        <parameters>$(arg simulation_controllers)</parameters>
+        <controller_manager_node_name>controller_manager</controller_manager_node_name>
+      </plugin>
+    </gazebo>
+  </xacro:if>
 </robot>
